File: eagle pcb v001/v1.brd (EAGLE design)
At the start: 40.3 x 14 mm, 6 parts

Commit message: nothing really.
resistor size double check. it was fine..
Parts:
- R1: device adafruit:0204/7 -> resistor:0204/7
Changed lines of the file:
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@@
 <element name="I2C" library="adafruit" package="1X04-CLEANBIG" value="1X4-CLEANBIG" x="21.59" y="1.27" rot="R180"/>
 <element name="PWR/BUZZER" library="adafruit" package="1X03-CLEANBIG" value="" x="21.59" y="12.7" rot="R180"/>
-<element name="R1" library="adafruit" package="0204/7" value="" x="15.24" y="8.89" rot="R90"/>
+<element name="R1" library="resistor" package="0204/7" value="" x="15.24" y="8.89" rot="R90"/>
 <element name="TINY" library="Atmel_By_element14_Batch_1-00" package="DIP254P762X533-8" value="ATTINY85-20PU" x="12.7" y="2.54">
 <attribute name="OC_FARNELL" value="1455162" x="12.7" y="2.54" size="1.778" layer="27" display="off"/>
